Commit message: remove redundant / unused assets

File: robosuite/models/assets/bullet_data/sawyer_description/urdf/sawyer_arm.urdf (robot description, URDF)
Before this commit: robot sawyer, 8 links, 7 joints
Links:
- link right_arm_base_link: geometry collision cylinder length=0.24 radius=0.08; visual mesh filename=package://sawyer_description/meshes/base.DAE
- link right_l0: geometry collision sphere radius=0.07; visual mesh filename=package://sawyer_description/meshes/l0.DAE
- link right_l1: geometry collision sphere radius=0.07; visual mesh filename=package://sawyer_description/meshes/l1.DAE
- link right_l2: geometry collision cylinder length=0.35 radius=0.06; visual mesh filename=package://sawyer_description/meshes/l2.DAE
- link right_l3: geometry collision sphere radius=0.06; visual mesh filename=package://sawyer_description/meshes/l3.DAE
- link right_l4: geometry collision cylinder length=0.36 radius=0.045; visual mesh filename=package://sawyer_description/meshes/l4.DAE
- link right_l5: geometry collision sphere radius=0.06; visual mesh filename=package://sawyer_description/meshes/l5.STL
- link right_l6: geometry collision cylinder length=0.05 radius=0.065; visual mesh filename=package://sawyer_description/meshes/l6.STL
