Commit message: updating cases

File: robosuite/models/assets/bullet_data/baxter_description/urdf/baxter_arm.urdf (robot description, URDF)
Before this commit: robot baxter, 49 links, 48 joints
Links:
- link head: geometry collision sphere radius=0.001; visual mesh filename=package://baxter_description/meshes/head/H0.dae
- link left_lower_elbow: geometry collision cylinder length=0.10 radius=0.06; visual mesh filename=package://baxter_description/meshes/lower_elbow/E1.dae
- link left_lower_forearm: geometry collision cylinder length=0.10 radius=0.06; visual mesh filename=package://baxter_description/meshes/lower_forearm/W1.dae
- link left_lower_shoulder: geometry collision cylinder length=0.12 radius=0.06; visual mesh filename=package://baxter_description/meshes/lower_shoulder/S1.dae
- link left_upper_elbow: geometry collision cylinder length=0.107 radius=0.06; visual mesh filename=package://baxter_description/meshes/upper_elbow/E0.dae
- link left_upper_forearm: geometry collision cylinder length=0.088 radius=0.06; visual mesh filename=package://baxter_description/meshes/upper_forearm/W0.dae
- link left_upper_shoulder: geometry collision cylinder length=0.2722 radius=0.06; visual mesh filename=package://baxter_description/meshes/upper_shoulder/S0.dae
- link left_wrist: geometry collision cylinder length=0.165 radius=0.06; visual mesh filename=package://baxter_description/meshes/wrist/W2.dae
- link pedestal: geometry visual mesh filename=package://baxter_description/meshes/base/PEDESTAL.dae
- link right_lower_elbow: geometry collision cylinder length=0.10 radius=0.06; visual mesh filename=package://baxter_description/meshes/lower_elbow/E1.dae
- link right_lower_forearm: geometry collision cylinder length=0.10 radius=0.06; visual mesh filename=package://baxter_description/meshes/lower_forearm/W1.dae
- link right_lower_shoulder: geometry collision cylinder length=0.12 radius=0.06; visual mesh filename=package://baxter_description/meshes/lower_shoulder/S1.dae
- link right_upper_elbow: geometry collision cylinder length=0.107 radius=0.06; visual mesh filename=package://baxter_description/meshes/upper_elbow/E0.dae
- link right_upper_forearm: geometry collision cylinder length=0.088 radius=0.06; visual mesh filename=package://baxter_description/meshes/upper_forearm/W0.dae
- link right_upper_shoulder: geometry collision cylinder length=0.2722 radius=0.06; visual mesh filename=package://baxter_description/meshes/upper_shoulder/S0.dae
- link right_wrist: geometry collision cylinder length=0.165 radius=0.06; visual mesh filename=package://baxter_description/meshes/wrist/W2.dae
- link screen: geometry collision sphere radius=0.001; visual mesh filename=package://baxter_description/meshes/head/H1.dae
- link torso: geometry visual mesh filename=package://baxter_description/meshes/torso/base_link.dae

File: robosuite/models/assets/bullet_data/sawyer_description/urdf/sawyer_arm.urdf (robot description, URDF)
Before this commit: robot sawyer, 8 links, 7 joints
Links:
- link right_arm_base_link: geometry collision cylinder length=0.24 radius=0.08; visual mesh filename=package://sawyer_description/meshes/base.dae
- link right_l0: geometry collision sphere radius=0.07; visual mesh filename=package://sawyer_description/meshes/l0.dae
- link right_l1: geometry collision sphere radius=0.07; visual mesh filename=package://sawyer_description/meshes/l1.dae
- link right_l2: geometry collision cylinder length=0.35 radius=0.06; visual mesh filename=package://sawyer_description/meshes/l2.dae
- link right_l3: geometry collision sphere radius=0.06; visual mesh filename=package://sawyer_description/meshes/l3.dae
- link right_l4: geometry collision cylinder length=0.36 radius=0.045; visual mesh filename=package://sawyer_description/meshes/l4.dae
- link right_l5: geometry collision sphere radius=0.06; visual mesh filename=package://sawyer_description/meshes/l5.stl
- link right_l6: geometry collision cylinder length=0.05 radius=0.065; visual mesh filename=package://sawyer_description/meshes/l6.stl
